File: schematic/spartan3.original/spartan3/spartan3.kicad_sch (KiCad schematic)
At the start: 208 parts

Commit message: Schematic :: LEDs polarity fixed/Power LED added
Parts:
- added D_vcc_0: LED_Small, symbol Device:LED_Small
- added R_vcc_0: 100R, symbol Device:R_US
Connections:
- net GND: now also R_vcc_0.2
- net VCC: now also D_in_bus1_one_0.2 (A), D_vcc_0.2 (A); no longer D_in_bus1_one_0.1 (K)
- net in_bus1: now also D_in_bus1_one_0.1 (K); no longer D_in_bus1_one_0.2 (A)
- net out_acc_r: now also D_out_acc_r_0.2 (A); no longer D_out_acc_r_0.1 (K)
- net out_acc_w: now also D_out_acc_w_0.2 (A); no longer D_out_acc_w_0.1 (K)
- net out_bus1: now also D_out_bus1_0.2 (A); no longer D_out_bus1_0.1 (K)
- net out_can_read: now also D_out_can_read_0.2 (A); no longer D_out_can_read_0.1 (K)
- net out_can_write: now also D_out_can_write_0.2 (A); no longer D_out_can_write_0.1 (K)
- net out_clk_internal: now also D_out_clk_internal_0.2 (A); no longer D_out_clk_internal_0.1 (K)
- net out_clkc: now also D_out_clkc_0.2 (A); no longer D_out_clkc_0.1 (K)
- net out_clkr: now also D_out_clkr_0.2 (A); no longer D_out_clkr_0.1 (K)
- net out_clkw: now also D_out_clkw_0.2 (A); no longer D_out_clkw_0.1 (K)
- net out_flags_C_out: now also D_out_flags_C_out_0.2 (A); no longer D_out_flags_C_out_0.1 (K)
- net out_flags_eq: now also D_out_flags_eq_0.2 (A); no longer D_out_flags_eq_0.1 (K)
- net out_flags_gt: now also D_out_flags_gt_0.2 (A); no longer D_out_flags_gt_0.1 (K)
- net out_flags_w: now also D_out_flags_w_0.2 (A); no longer D_out_flags_w_0.1 (K)
- net out_flags_z: now also D_out_flags_z_0.2 (A); no longer D_out_flags_z_0.1 (K)
- net out_iar_r: now also D_out_iar_r_0.2 (A); no longer D_out_iar_r_0.1 (K)
- net out_iar_w: now also D_out_iar_w_0.2 (A); no longer D_out_iar_w_0.1 (K)
- net out_ir_w: now also D_out_ir_w_0.2 (A); no longer D_out_ir_w_0.1 (K)
- net out_is_bus1_w: now also D_out_is_bus1_w_0.2 (A); no longer D_out_is_bus1_w_0.1 (K)
- net out_r0_r: now also D_out_r0_r_0.2 (A); no longer D_out_r0_r_0.1 (K)
- net out_r0_w: now also D_out_r0_w_0.2 (A); no longer D_out_r0_w_0.1 (K)
- net out_r1_r: now also D_out_r1_r_0.2 (A); no longer D_out_r1_r_0.1 (K)
- net out_r1_w: now also D_out_r1_w_0.2 (A); no longer D_out_r1_w_0.1 (K)
- net out_r2_r: now also D_out_r2_r_0.2 (A); no longer D_out_r2_r_0.1 (K)
- net out_r2_w: now also D_out_r2_w_0.2 (A); no longer D_out_r2_w_0.1 (K)
- net out_r3_r: now also D_out_r3_r_0.2 (A); no longer D_out_r3_r_0.1 (K)
- net out_r3_w: now also D_out_r3_w_0.2 (A); no longer D_out_r3_w_0.1 (K)
- net out_ram_a_w: now also D_out_ram_a_w_0.2 (A); no longer D_out_ram_a_w_0.1 (K)
- net out_ram_r: now also D_out_ram_r_0.2 (A); no longer D_out_ram_r_0.1 (K)
- net out_ram_w: now also D_out_ram_w_0.2 (A); no longer D_out_ram_w_0.1 (K)
- net out_s1: now also D_out_s1_0.2 (A); no longer D_out_s1_0.1 (K)
- net out_s2: now also D_out_s2_0.2 (A); no longer D_out_s2_0.1 (K)
- net out_s3: now also D_out_s3_0.2 (A); no longer D_out_s3_0.1 (K)
- net out_s4: now also D_out_s4_0.2 (A); no longer D_out_s4_0.1 (K)
- net out_s5: now also D_out_s5_0.2 (A); no longer D_out_s5_0.1 (K)
- net out_s6: now also D_out_s6_0.2 (A); no longer D_out_s6_0.1 (K)
- net out_sysbus_0: now also D_out_sysbus_0.2 (A); no longer D_out_sysbus_0.1 (K)
- net out_sysbus_1: now also D_out_sysbus_1.2 (A); no longer D_out_sysbus_1.1 (K)
- net out_sysbus_2: now also D_out_sysbus_2.2 (A); no longer D_out_sysbus_2.1 (K)
- net out_sysbus_3: now also D_out_sysbus_3.2 (A); no longer D_out_sysbus_3.1 (K)
- net out_sysbus_4: now also D_out_sysbus_4.2 (A); no longer D_out_sysbus_4.1 (K)
- net out_sysbus_5: now also D_out_sysbus_5.2 (A); no longer D_out_sysbus_5.1 (K)
- net out_sysbus_6: now also D_out_sysbus_6.2 (A); no longer D_out_sysbus_6.1 (K)
- net out_sysbus_7: now also D_out_sysbus_7.2 (A); no longer D_out_sysbus_7.1 (K)
- net out_temp_w: now also D_out_temp_w_0.2 (A); no longer D_out_temp_w_0.1 (K)
- net at R_out_sysbus_3.1: now also D_out_sysbus_3.1 (K); no longer D_out_sysbus_3.2 (A)
- net at R_out_can_read_0.1: now also D_out_can_read_0.1 (K); no longer D_out_can_read_0.2 (A)
- net at R_out_s1_0.1: now also D_out_s1_0.1 (K); no longer D_out_s1_0.2 (A)
- net at R_out_sysbus_2.1: now also D_out_sysbus_2.1 (K); no longer D_out_sysbus_2.2 (A)
- net at R_out_flags_z_0.1: now also D_out_flags_z_0.1 (K); no longer D_out_flags_z_0.2 (A)
- net at R_out_r3_w_0.1: now also D_out_r3_w_0.1 (K); no longer D_out_r3_w_0.2 (A)
- net at R_out_r3_r_0.1: now also D_out_r3_r_0.1 (K); no longer D_out_r3_r_0.2 (A)
- net at R_out_sysbus_0.1: now also D_out_sysbus_0.1 (K); no longer D_out_sysbus_0.2 (A)
- net at R_out_sysbus_4.1: now also D_out_sysbus_4.1 (K); no longer D_out_sysbus_4.2 (A)
- net at R_out_temp_w_0.1: now also D_out_temp_w_0.1 (K); no longer D_out_temp_w_0.2 (A)
- net at R_out_clkc_0.1: now also D_out_clkc_0.1 (K); no longer D_out_clkc_0.2 (A)
- net at R_out_clk_internal_0.1: now also D_out_clk_internal_0.1 (K); no longer D_out_clk_internal_0.2 (A)
- net at R_out_s3_0.1: now also D_out_s3_0.1 (K); no longer D_out_s3_0.2 (A)
- net at R_out_s2_0.1: now also D_out_s2_0.1 (K); no longer D_out_s2_0.2 (A)
- net at R_out_iar_r_0.1: now also D_out_iar_r_0.1 (K); no longer D_out_iar_r_0.2 (A)
- net at R_out_s4_0.1: now also D_out_s4_0.1 (K); no longer D_out_s4_0.2 (A)
- net at R_out_r1_r_0.1: now also D_out_r1_r_0.1 (K); no longer D_out_r1_r_0.2 (A)
- net at R_out_ir_w_0.1: now also D_out_ir_w_0.1 (K); no longer D_out_ir_w_0.2 (A)
- net at R_out_r0_w_0.1: now also D_out_r0_w_0.1 (K); no longer D_out_r0_w_0.2 (A)
- net at R_out_r2_r_0.1: now also D_out_r2_r_0.1 (K); no longer D_out_r2_r_0.2 (A)
- net at R_out_ram_a_w_0.1: now also D_out_ram_a_w_0.1 (K); no longer D_out_ram_a_w_0.2 (A)
- net at R_out_is_bus1_w_0.1: now also D_out_is_bus1_w_0.1 (K); no longer D_out_is_bus1_w_0.2 (A)
- net at R_out_flags_eq_0.1: now also D_out_flags_eq_0.1 (K); no longer D_out_flags_eq_0.2 (A)
- net at R_out_can_write_0.1: now also D_out_can_write_0.1 (K); no longer D_out_can_write_0.2 (A)
- net at R_out_r2_w_0.1: now also D_out_r2_w_0.1 (K); no longer D_out_r2_w_0.2 (A)
- net at R_out_clkw_0.1: now also D_out_clkw_0.1 (K); no longer D_out_clkw_0.2 (A)
- net at R_out_iar_w_0.1: now also D_out_iar_w_0.1 (K); no longer D_out_iar_w_0.2 (A)
- net at R_out_ram_w_0.1: now also D_out_ram_w_0.1 (K); no longer D_out_ram_w_0.2 (A)
- net at R_out_s5_0.1: now also D_out_s5_0.1 (K); no longer D_out_s5_0.2 (A)
- net at R_out_acc_w_0.1: now also D_out_acc_w_0.1 (K); no longer D_out_acc_w_0.2 (A)
- net at R_out_ram_r_0.1: now also D_out_ram_r_0.1 (K); no longer D_out_ram_r_0.2 (A)
- net at R_out_flags_w_0.1: now also D_out_flags_w_0.1 (K); no longer D_out_flags_w_0.2 (A)
- net at R_out_sysbus_5.1: now also D_out_sysbus_5.1 (K); no longer D_out_sysbus_5.2 (A)
- net at R_out_sysbus_7.1: now also D_out_sysbus_7.1 (K); no longer D_out_sysbus_7.2 (A)
- net at R_out_sysbus_6.1: now also D_out_sysbus_6.1 (K); no longer D_out_sysbus_6.2 (A)
- net at R_out_r1_w_0.1: now also D_out_r1_w_0.1 (K); no longer D_out_r1_w_0.2 (A)
- net at R_out_flags_C_out_0.1: now also D_out_flags_C_out_0.1 (K); no longer D_out_flags_C_out_0.2 (A)
- net at R_out_r0_r_0.1: now also D_out_r0_r_0.1 (K); no longer D_out_r0_r_0.2 (A)
- net at R_out_sysbus_1.1: now also D_out_sysbus_1.1 (K); no longer D_out_sysbus_1.2 (A)
- net at R_out_acc_r_0.1: now also D_out_acc_r_0.1 (K); no longer D_out_acc_r_0.2 (A)
- net at R_out_s6_0.1: now also D_out_s6_0.1 (K); no longer D_out_s6_0.2 (A)
- net at R_out_flags_gt_0.1: now also D_out_flags_gt_0.1 (K); no longer D_out_flags_gt_0.2 (A)
- net at R_out_bus1_0.1: now also D_out_bus1_0.1 (K); no longer D_out_bus1_0.2 (A)
- net at R_out_clkr_0.1: now also D_out_clkr_0.1 (K); no longer D_out_clkr_0.2 (A)
- new net: D_vcc_0.1 (K), R_vcc_0.1
Other:
- moved on the sheet: D_in_bus1_one_0, D_out_acc_r_0, D_out_acc_w_0, D_out_bus1_0, D_out_can_read_0, D_out_can_write_0, D_out_clk_internal_0, D_out_clkc_0, D_out_clkr_0, D_out_clkw_0, D_out_flags_C_out_0, D_out_flags_eq_0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

Commit message: Schematics :: footprints partially assigned
Parts:
- C_clk_0, C_clk_1, C_eeprom_vcc_0: footprint (none) -> Capacitor_SMD:C_0805_2012Metric_Pad1.18x1.45mm_HandSolder
- D1: renamed from D?; footprint (none) -> LED_SMD:LED_0805_2012Metric_Pad1.15x1.40mm_HandSolder
- D_in_acc_r_0, D_in_acc_w_0, D_in_bus1_one_0, D_in_bus1_ps_0, D_in_clk_manual_0, D_in_iar_r_0, D_in_iar_w_0, D_in_ir_r_0, D_in_ir_w_0, D_in_is_bus1_w_0, D_in_is_clk_external_0, D_in_is_clk_high_0, D_in_is_clk_low_0, D_in_is_clk_manual_0, D_in_is_clk_veryhigh_0, D_in_manual_input_r_0, D_in_r0_r_0, D_in_r0_w_0, D_in_r1_r_0, D_in_r1_w_0, D_in_r2_r_0, D_in_r2_w_0, D_in_r3_r_0, D_in_r3_w_0, D_in_ram_a_w_0, D_in_ram_r_0, D_in_ram_w_0, D_in_read_reg_en_0, D_in_temp_w_0, D_in_write_reg_en_0, D_out_acc_r_0, D_out_acc_w_0, D_out_bus1_0, D_out_can_read_0, D_out_can_write_0, D_out_clk_internal_0, D_out_clkc_0, D_out_clkr_0, D_out_clkw_0, D_out_flags_C_out_0, D_out_flags_eq_0, D_out_flags_gt_0, D_out_flags_w_0, D_out_flags_z_0, D_out_iar_r_0, D_out_iar_w_0, D_out_ir_w_0, D_out_is_bus1_w_0, D_out_r0_r_0, D_out_r0_w_0, D_out_r1_r_0, D_out_r1_w_0, D_out_r2_r_0, D_out_r2_w_0, D_out_r3_r_0, D_out_r3_w_0, D_out_ram_a_w_0, D_out_ram_r_0, D_out_ram_w_0, D_out_s1_0, D_out_s2_0, D_out_s3_0, D_out_s4_0, D_out_s5_0, D_out_s6_0, D_out_sysbus_0, D_out_sysbus_1, D_out_sysbus_2, D_out_sysbus_3, D_out_sysbus_4, D_out_sysbus_5, D_out_sysbus_6, D_out_sysbus_7, D_out_temp_w_0, D_vcc_0: footprint (none) -> LED_SMD:LED_0805_2012Metric_Pad1.15x1.40mm_HandSolder
- F_pwr_0: footprint (none) -> Fuse:Fuse_0805_2012Metric_Pad1.15x1.40mm_HandSolder
- J_JTAG_0: footprint (none) -> Connector_IDC:IDC-Header_2x05_P2.54mm_Vertical
- J_pwr_0: footprint (none) -> Connector_USB:USB_A_Molex_67643_Horizontal
- L_clk_0: footprint (none) -> Inductor_SMD:L_0805_2012Metric_Pad1.05x1.20mm_HandSolder
- R1: renamed from R?; footprint (none) -> Resistor_SMD:R_0805_2012Metric_Pad1.20x1.40mm_HandSolder
- R_JTAG_TCK_0, R_JTAG_TDI_0, R_JTAG_TDO_0, R_JTAG_TMS_0, R__eeprom_dq1_0, R_clk_oe_0, R_clk_out_0, R_eeprom_hold_0, R_eeprom_s_0, R_eeprom_w_0, R_in_acc_r_0, R_in_acc_w_0, R_in_bus1_0, R_in_clk_manual_0, R_in_iar_r_0, R_in_iar_w_0, R_in_ir_r_0, R_in_ir_w_0, R_in_is_bus1_w_0, R_in_is_clk_external_0, R_in_is_clk_high_0, R_in_is_clk_low_0, R_in_is_clk_manual_0, R_in_is_clk_veryhigh_0, R_in_manual_input_o_0, R_in_manual_input_o_1, R_in_manual_input_o_2, R_in_manual_input_o_3, R_in_manual_input_o_4, R_in_manual_input_o_5, R_in_manual_input_o_6, R_in_manual_input_o_7, R_in_manual_input_r_0, R_in_r0_r_0, R_in_r0_w_0, R_in_r1_r_0, R_in_r1_w_0, R_in_r2_r_0, R_in_r2_w_0, R_in_r3_r_0, R_in_r3_w_0, R_in_ram_a_w_0, R_in_ram_r_0, R_in_ram_w_0, R_in_read_reg_en_0, R_in_temp_w_0, R_in_write_reg_en_0, R_out_acc_r_0, R_out_acc_w_0, R_out_bus1_0, R_out_can_read_0, R_out_can_write_0, R_out_clk_internal_0, R_out_clkc_0, R_out_clkr_0, R_out_clkw_0, R_out_flags_C_out_0, R_out_flags_eq_0, R_out_flags_gt_0, R_out_flags_w_0, R_out_flags_z_0, R_out_iar_r_0, R_out_iar_w_0, R_out_ir_w_0, R_out_is_bus1_w_0, R_out_r0_r_0, R_out_r0_w_0, R_out_r1_r_0, R_out_r1_w_0, R_out_r2_r_0, R_out_r2_w_0, R_out_r3_r_0, R_out_r3_w_0, R_out_ram_a_w_0, R_out_ram_r_0, R_out_ram_w_0, R_out_s1_0, R_out_s2_0, R_out_s3_0, R_out_s4_0, R_out_s5_0, R_out_s6_0, R_out_sysbus_0, R_out_sysbus_1, R_out_sysbus_2, R_out_sysbus_3, R_out_sysbus_4, R_out_sysbus_5, R_out_sysbus_6, R_out_sysbus_7, R_out_temp_w_0, R_vcc_0: footprint (none) -> Resistor_SMD:R_0805_2012Metric_Pad1.20x1.40mm_HandSolder
- SW_in_acc_w_0, SW_in_bus1_0, SW_in_clk_manual_0, SW_in_iar_w_0, SW_in_ir_w_0, SW_in_is_bus1_w_0, SW_in_r0_w_0, SW_in_r1_w_0, SW_in_r2_w_0, SW_in_r3_w_0, SW_in_ram_a_w_0, SW_in_ram_w_0, SW_in_read_reg_en_0, SW_in_temp_w_0, SW_in_write_reg_en_0, SW_pwr_0: footprint (none) -> Button_Switch_THT:SW_Push_2P2T_Toggle_CK_PVA2OAH5xxxxxxV2
- SW_in_manual_input_o_0, SW_in_manual_input_o_1, SW_in_manual_input_o_2, SW_in_manual_input_o_3, SW_in_manual_input_o_4, SW_in_manual_input_o_5, SW_in_manual_input_o_6, SW_in_manual_input_o_7: footprint (none) -> Button_Switch_THT:SW_Slide_1P2T_CK_OS102011MS2Q
- U2: renamed from U?; footprint TQ144 -> Package_QFP:TQFP-144_20x20mm_P0.5mm
- U_eeprom_0: footprint (none) -> Package_SO:SO-8_5.3x6.2mm_P1.27mm
- gave numbers to parts that had none: 1

Commit message: Schematics :: SW Rotary 12 footprint added
Parts:
- SW_read_register_0: footprint (none) -> SR26 1-1-12P:SR26 1-1-12P
- U1_clk_select_0: footprint (none) -> Connector_PinHeader_1.27mm:PinHeader_1x07_P1.27mm_Vertical
- U_eeprom_0: footprint Package_SO:SO-8_5.3x6.2mm_P1.27mm -> Package_SO:SOIC-8-1EP_3.9x4.9mm_P1.27mm_EP2.29x3mm
Changed lines of the file:
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@@
     (property "Reference" "SW_read_register_0" (id 0) (at 521.0175 128.5072 0))
     (property "Value" "SW_Rotary12" (id 1) (at 521.0175 131.0441 0))
-    (property "Footprint" "" (id 2) (at 523.24 165.1 0)
+    (property "Footprint" "SR26 1-1-12P:SR26 1-1-12P" (id 2) (at 523.24 165.1 0)
       (effects (font (size 1.27 1.27)) hide)
     )
@@
       (effects (font (size 1.27 1.27)) (justify right))
     )
-    (property "Footprint" "" (id 2) (at 344.17 394.97 0)
+    (property "Footprint" "Connector_PinHeader_1.27mm:PinHeader_1x07_P1.27mm_Vertical" (id 2) (at 344.17 394.97 0)
       (effects (font (size 1.27 1.27)) hide)
     )
@@
     (property "Reference" "U_eeprom_0" (id 0) (at 850.9 353.221 0))
     (property "Value" "M25P16-VMN3PB" (id 1) (at 850.9 355.7579 0))
-    (property "Footprint" "Package_SO:SO-8_5.3x6.2mm_P1.27mm" (id 2) (at 850.9 354.33 0)
+    (property "Footprint" "Package_SO:SOIC-8-1EP_3.9x4.9mm_P1.27mm_EP2.29x3mm" (id 2) (at 850.9 354.33 0)
       (effects (font (size 1.27 1.27)) hide)
     )
@@
     )
     (path "/03864d95-12e9-4ac3-8fe8-12f816999570"
-      (reference "SW_read_register_0") (unit 1) (value "SW_Rotary12") (footprint "")
+      (reference "SW_read_register_0") (unit 1) (value "SW_Rotary12") (footprint "SR26 1-1-12P:SR26 1-1-12P")
     )
     (path "/3dc17902-13b6-4e7e-8b7b-bbfdc1838232"
-      (reference "U1_clk_select_0") (unit 1) (value "SPFT_Sliding_Switch-dynacore") (footprint "")
+      (reference "U1_clk_select_0") (unit 1) (value "SPFT_Sliding_Switch-dynacore") (footprint "Connector_PinHeader_1.27mm:PinHeader_1x07_P1.27mm_Vertical")
     )
     (path "/1fb658dc-8205-48c7-9b5e-baf76f32a857"
@@
     )
     (path "/8be28da1-efdd-4074-85b4-c20318b00a07"
-      (reference "U_eeprom_0") (unit 1) (value "M25P16-VMN3PB") (footprint "Package_SO:SO-8_5.3x6.2mm_P1.27mm")
+      (reference "U_eeprom_0") (unit 1) (value "M25P16-VMN3PB") (footprint "Package_SO:SOIC-8-1EP_3.9x4.9mm_P1.27mm_EP2.29x3mm")
     )
     (path "/c3fd6b01-2f54-4af3-b308-6167cf316338"

Commit message: Schematics :: JTAG/SPST/SPDT updated
Parts:
- removed D1: LED_Small, LED_SMD:LED_0805_2012Metric_Pad1.15x1.40mm_HandSolder, symbol Device:LED_Small
- removed J_JTAG_0: Conn_ARM_JTAG_SWD_10, Connector_IDC:IDC-Header_2x05_P2.54mm_Vertical, symbol Connector:Conn_ARM_JTAG_SWD_10
- removed R1: R_US, Resistor_SMD:R_0805_2012Metric_Pad1.20x1.40mm_HandSolder, symbol Device:R_US
- added P_JTAG_0: Xilinx_JTAG, Connector_IDC:IDC-Header_2x07-1MP_P2.54mm_Latch_Vertical, symbol sliders:Xilinx_JTAG
- D_out_sysbus_0, D_out_sysbus_1, D_out_sysbus_2, D_out_sysbus_3, D_out_sysbus_4, D_out_sysbus_5, D_out_sysbus_6, D_out_sysbus_7: footprint LED_SMD:LED_0805_2012Metric_Pad1.15x1.40mm_HandSolder -> SW_SPDT_small:SW_SPDT_Small
- SW_in_clk_manual_0: footprint Button_Switch_THT:SW_Push_2P2T_Toggle_CK_PVA2OAH5xxxxxxV2 -> SPST_square:SPST_Square
- U1_clk_select_0: footprint Connector_PinHeader_1.27mm:PinHeader_1x07_P1.27mm_Vertical -> SW_Sliding_5Pos:SW_Sliding_5Pos
Connections:
- net GND: now also P_JTAG_0.1 (GND), P_JTAG_0.11 (GND), P_JTAG_0.13 (GND), P_JTAG_0.3 (GND), P_JTAG_0.5 (GND), P_JTAG_0.7 (GND), P_JTAG_0.9 (GND)
- net VCC_banks: now also P_JTAG_0.2 (VCC_ref)
- net at R_JTAG_TCK_0.1: now also P_JTAG_0.6 (TCK)
- net at R_JTAG_TMS_0.1: now also P_JTAG_0.4 (TMS)
- net at R_JTAG_TDO_0.1: now also P_JTAG_0.8 (TDO)
- net at R_JTAG_TDI_0.1: now also P_JTAG_0.10 (TDI)
Other:
- note removed: "Read"
