File: schematic/spartan3.original/spartan3/spartan3.kicad_pcb (KiCad board)
At the start: 2 copper layers, 200 x 160 mm, 219 parts, among them U1_clk_select_0 SPFT_Sliding_Switch-dynacore, U2 XC3S250E-4TQG144C

Commit message: Schematics :: updated / PCB layout :: updated
Parts:
- added R_d_in_acc_w_0: 100R, Resistor_SMD:R_0805_2012Metric_Pad1.20x1.40mm_HandSolder, F.Cu at (205.7, 137.2)
- added R_d_in_bus1_one_0: 100R, Resistor_SMD:R_0805_2012Metric_Pad1.20x1.40mm_HandSolder, F.Cu at (55.9, 104.1)
- added R_d_in_bus1_ps_0: 100R, Resistor_SMD:R_0805_2012Metric_Pad1.20x1.40mm_HandSolder, F.Cu at (54.3, 96.5)
- added R_d_in_clk_manual_0: 100R, Resistor_SMD:R_0805_2012Metric_Pad1.20x1.40mm_HandSolder, F.Cu at (5.08, 162.6)
- added R_d_in_iar_w_0: 100R, Resistor_SMD:R_0805_2012Metric_Pad1.20x1.40mm_HandSolder, F.Cu at (221.0, 177.8)
- added R_d_in_ir_w_0: 100R, Resistor_SMD:R_0805_2012Metric_Pad1.20x1.40mm_HandSolder, F.Cu at (208.3, 157.5)
- added R_d_in_is_bus1_w_0: 100R, Resistor_SMD:R_0805_2012Metric_Pad1.20x1.40mm_HandSolder, F.Cu at (53.3, 86.4)
- added R_d_in_is_clk_external_0: 100R, Resistor_SMD:R_0805_2012Metric_Pad1.20x1.40mm_HandSolder, F.Cu at (82.3, 137.2)
- added R_d_in_is_clk_high_0: 100R, Resistor_SMD:R_0805_2012Metric_Pad1.20x1.40mm_HandSolder, F.Cu at (82.3, 152.4)
- added R_d_in_is_clk_low_0: 100R, Resistor_SMD:R_0805_2012Metric_Pad1.20x1.40mm_HandSolder, F.Cu at (82.3, 147.3)
- added R_d_in_is_clk_manual_0: 100R, Resistor_SMD:R_0805_2012Metric_Pad1.20x1.40mm_HandSolder, F.Cu at (82.3, 157.5)
- added R_d_in_is_clk_veryhigh_0: 100R, Resistor_SMD:R_0805_2012Metric_Pad1.20x1.40mm_HandSolder, F.Cu at (81.3, 142.2)
- added R_d_in_r0_w_0: 100R, Resistor_SMD:R_0805_2012Metric_Pad1.20x1.40mm_HandSolder, F.Cu at (209.3, 167.6)
- added R_d_in_r1_w_0: 100R, Resistor_SMD:R_0805_2012Metric_Pad1.20x1.40mm_HandSolder, F.Cu at (208.3, 142.2)
- added R_d_in_r2_w_0: 100R, Resistor_SMD:R_0805_2012Metric_Pad1.20x1.40mm_HandSolder, F.Cu at (208.3, 162.6)
- added R_d_in_r3_w_0: 100R, Resistor_SMD:R_0805_2012Metric_Pad1.20x1.40mm_HandSolder, F.Cu at (208.3, 152.4)
- added R_d_in_ram_a_w_0: 100R, Resistor_SMD:R_0805_2012Metric_Pad1.20x1.40mm_HandSolder, F.Cu at (221.0, 172.7)
- added R_d_in_ram_w_0: 100R, Resistor_SMD:R_0805_2012Metric_Pad1.20x1.40mm_HandSolder, F.Cu at (206.7, 132.1)
- added R_d_in_read_reg_en_0: 100R, Resistor_SMD:R_0805_2012Metric_Pad1.20x1.40mm_HandSolder, F.Cu at (71.1, 30.5)
- added R_d_in_temp_w_0: 100R, Resistor_SMD:R_0805_2012Metric_Pad1.20x1.40mm_HandSolder, F.Cu at (208.3, 147.3)
- added R_d_in_write_reg_en_0: 100R, Resistor_SMD:R_0805_2012Metric_Pad1.20x1.40mm_HandSolder, F.Cu at (127.0, 25.4)
- moved D_in_write_reg_en_0 124.7 mm to (143.3, 35.6)
- moved R_in_write_reg_en_0 122.0 mm to (142.2, 30.5)
- moved R_out_can_read_0 27.8 mm to (26.4, 27.9)
- moved D_out_can_read_0 25.0 mm to (17.8, 27.9)
- moved D_in_is_bus1_w_0 23.4 mm to (52.3, 81.3)
- moved R_in_ram_r_0 5.68 mm to (68.6, 63.5)
Connections:
- D_in_acc_w_0 pad 2: VCC -> Net-(D_in_acc_w_0-Pad2)
- D_in_bus1_one_0 pad 2: VCC -> Net-(D_in_bus1_one_0-Pad2)
- D_in_bus1_ps_0 pad 1: GND -> Net-(D_in_bus1_ps_0-Pad1)
- D_in_clk_manual_0 pad 2: VCC -> Net-(D_in_clk_manual_0-Pad2)
- D_in_iar_w_0 pad 2: VCC -> Net-(D_in_iar_w_0-Pad2)
- D_in_ir_w_0 pad 2: VCC -> Net-(D_in_ir_w_0-Pad2)
- D_in_is_bus1_w_0 pad 2: VCC -> Net-(D_in_is_bus1_w_0-Pad2)
- D_in_is_clk_external_0 pad 2: VCC -> Net-(D_in_is_clk_external_0-Pad2)
- D_in_is_clk_high_0 pad 2: VCC -> Net-(D_in_is_clk_high_0-Pad2)
- D_in_is_clk_low_0 pad 2: VCC -> Net-(D_in_is_clk_low_0-Pad2)
- D_in_is_clk_manual_0 pad 2: VCC -> Net-(D_in_is_clk_manual_0-Pad2)
- D_in_is_clk_veryhigh_0 pad 2: VCC -> Net-(D_in_is_clk_veryhigh_0-Pad2)
- D_in_r0_w_0 pad 2: VCC -> Net-(D_in_r0_w_0-Pad2)
- D_in_r1_w_0 pad 2: VCC -> Net-(D_in_r1_w_0-Pad2)
- D_in_r2_w_0 pad 2: VCC -> Net-(D_in_r2_w_0-Pad2)
- D_in_r3_w_0 pad 2: VCC -> Net-(D_in_r3_w_0-Pad2)
- D_in_ram_a_w_0 pad 2: VCC -> Net-(D_in_ram_a_w_0-Pad2)
- D_in_ram_w_0 pad 2: VCC -> Net-(D_in_ram_w_0-Pad2)
- D_in_read_reg_en_0 pad 2: VCC -> Net-(D_in_read_reg_en_0-Pad2)
- D_in_temp_w_0 pad 2: VCC -> Net-(D_in_temp_w_0-Pad2)
- D_in_write_reg_en_0 pad 2: VCC -> Net-(D_in_write_reg_en_0-Pad2)

Commit message: PCB layout :: updated
Parts:
- R_JTAG_TDI_0, U2, U_eeprom_0, U_pwr_vcc_banks_0, U_pwr_vcc_core_0, U_pwr_vcc_peripheral_0, X_clk_0: moved to F.Cu
- moved R_d_in_iar_w_0 185.4 mm to (99.1, 38.1)
- moved R_in_iar_w_0 178.5 mm to (94.0, 40.6)
- moved D_in_iar_w_0 172.7 mm to (94.0, 38.1)
- moved R_d_in_ram_a_w_0 155.5 mm to (99.1, 76.2)
- moved R_d_in_ir_w_0 152.7 mm to (99.1, 50.8)
- moved R_in_ram_a_w_0 148.0 mm to (94.0, 78.7)
- moved D_in_ir_w_0 147.3 mm to (94.0, 50.8)
- moved R_d_in_r0_w_0 143.8 mm to (125.5, 50.8)
- moved D_in_ram_a_w_0 140.1 mm to (94.0, 76.2)
- moved D_in_r0_w_0 139.5 mm to (119.4, 50.8)
- moved R_in_ir_w_0 138.6 mm to (94.0, 53.3)
- moved R_d_in_temp_w_0 137.7 mm to (124.5, 38.1)
- moved D_in_temp_w_0 134.9 mm to (117.9, 38.1)
- moved R_in_r0_w_0 132.0 mm to (119.4, 53.3)
- moved R_d_in_acc_w_0 129.6 mm to (99.1, 63.5)
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Other:
- board size 200 x 160 mm -> 214.6 x 160 mm

Commit message: PCB layout updated
Parts:
- moved R_out_acc_r_0 173.3 mm to (30.5, 109.2)
- moved D_out_acc_r_0 169.9 mm to (30.5, 106.7)
- moved R_out_ram_w_0 156.5 mm to (40.6, 116.8)
- moved D_out_ram_w_0 150.3 mm to (40.6, 114.3)
- moved R_out_acc_w_0 145.5 mm to (30.5, 116.8)
- moved D_out_acc_w_0 137.3 mm to (30.5, 114.3)
- moved D_out_r1_r_0 130.4 mm to (101.6, 106.7)
- moved R_out_r1_r_0 130.0 mm to (101.6, 109.2)
- moved R_out_ram_a_w_0 127.3 mm to (71.1, 116.8)
- moved D_out_ram_a_w_0 122.7 mm to (71.1, 114.3)
- moved R_out_ram_r_0 122.3 mm to (40.6, 109.2)
- moved R_out_iar_r_0 118.9 mm to (20.3, 109.2)
- moved R_out_iar_w_0 118.4 mm to (20.3, 116.8)
- moved D_out_ram_r_0 115.0 mm to (40.6, 106.7)
- moved R_out_temp_w_0 111.9 mm to (61.0, 116.8)
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
Commit message: PCB layout :: updated
Parts:
- moved R_in_is_bus1_w_0 28.4 mm to (44.2, 81.3)
- moved R_in_read_reg_en_0 25.9 mm to (45.7, 30.5)
- moved R_in_write_reg_en_0 23.4 mm to (99.1, 30.5)
- moved R_in_bus1_0 23.0 mm to (43.2, 91.4)
- moved R_d_in_none_r_0 20.9 mm to (34.0, 38.1)
- moved SW_in_bus1_0 20.5 mm to (53.0, 93.9)
- moved R_d_in_bus1_one_0 18.0 mm to (71.1, 94.0)
- moved R_reset_0 18.0 mm to (7.62, 111.8)
- moved D_in_is_bus1_w_0 16.4 mm to (55.8, 80.7)
- moved R_out_r3_r_0 16.1 mm to (106.6, 114.3)
- moved D_out_r3_r_0 15.9 mm to (106.6, 111.2)
- moved R_d_in_bus1_ps_0 15.9 mm to (70.1, 88.4)
- moved SW_in_write_reg_en_0 15.8 mm to (119.4, 32.9)
- moved R_out_r3_w_0 15.6 mm to (106.6, 121.9)
- moved R_d_in_is_bus1_w_0 15.5 mm to (55.8, 83.8)
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- renumbered R_out_acc_w_0 to locked
Other:
- board size 214.6 x 160 mm -> 215.9 x 160 mm
